File: thermistors.kicad_sch (KiCad schematic)
At the start: 5 parts, among them J3 THERM_1, J4 THERM_2

Commit message: schematic: Cleanup BOM
Parts:
- J3, J4: Dist (none) -> LCSC; Dist # (none) -> C495200; Mfr (none) -> JST; Mfr # (none) -> S20B-PUDSS-1(LF)(SN); Part Number S20B-PUDSS-1 -> (none); Role Thermistor connector -> (none)
- TH1, TH2, TH3: Dist (none) -> LCSC; Dist # (none) -> C525660; Mfr (none) -> Sunlord; Mfr # (none) -> SDNT1608X103F3435FTF; Part Number SDNT1608X103F3435FTF -> (none); Role On-board thermistor -> (none)
Changed lines of the file:
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@@
 			)
 		)
-		(property "Part Number" "S20B-PUDSS-1"
+		(property "Dist #" "C495200"
 			(at 139.7 69.85 0)
 			(effects
@@
 			)
 		)
-		(property "Role" "Thermistor connector"
+		(property "Mfr" "JST"
+			(at 139.7 69.85 0)
+			(effects
+				(font
+					(size 1.27 1.27)
+				)
+				(hide yes)
+			)
+		)
+		(property "Mfr #" "S20B-PUDSS-1(LF)(SN)"
+			(at 139.7 69.85 0)
+			(effects
+				(font
+					(size 1.27 1.27)
+				)
+				(hide yes)
+			)
+		)
+		(property "Dist" "LCSC"
 			(at 139.7 69.85 0)
 			(effects
@@
 			)
 		)
-		(property "Role" "On-board thermistor"
+		(property "Dist #" "C525660"
 			(at 60.96 63.5 0)
 			(effects
@@
 			)
 		)
-		(property "Part Number" " SDNT1608X103F3435FTF"
+		(property "Mfr" " Sunlord"
+			(at 60.96 63.5 0)
+			(effects
+				(font
+					(size 1.27 1.27)
+				)
+				(hide yes)
+			)
+		)
+		(property "Mfr #" "SDNT1608X103F3435FTF"
+			(at 60.96 63.5 0)
+			(effects
+				(font
+					(size 1.27 1.27)
+				)
+				(hide yes)
+			)
+		)
+		(property "Dist" "LCSC"
 			(at 60.96 63.5 0)
 			(effects
@@
 			)
 		)
-		(property "Part Number" "S20B-PUDSS-1"
-			(at 139.7 95.25 0)
-			(effects
-				(font
-					(size 1.27 1.27)
-				)
-				(hide yes)
-			)
-		)
-		(property "Role" "Thermistor connector"
+		(property "Dist #" "C495200"
+			(at 139.7 95.25 0)
+			(effects
+				(font
+					(size 1.27 1.27)
+				)
+				(hide yes)
+			)
+		)
+		(property "Mfr" "JST"
+			(at 139.7 95.25 0)
+			(effects
+				(font
+					(size 1.27 1.27)
+				)
+				(hide yes)
+			)
+		)
+		(property "Mfr #" "S20B-PUDSS-1(LF)(SN)"
+			(at 139.7 95.25 0)
+			(effects
+				(font
+					(size 1.27 1.27)
+				)
+				(hide yes)
+			)
+		)
+		(property "Dist" "LCSC"
 			(at 139.7 95.25 0)
 			(effects
@@
 			)
 		)
-		(property "Role" "On-board thermistor"
+		(property "Dist #" "C525660"
 			(at 60.96 50.8 0)
 			(effects
@@
 			)
 		)
-		(property "Part Number" " SDNT1608X103F3435FTF"
+		(property "Mfr" " Sunlord"
+			(at 60.96 50.8 0)
+			(effects
+				(font
+					(size 1.27 1.27)
+				)
+				(hide yes)
+			)
+		)
+		(property "Mfr #" "SDNT1608X103F3435FTF"
+			(at 60.96 50.8 0)
+			(effects
+				(font
+					(size 1.27 1.27)
+				)
+				(hide yes)
+			)
+		)
+		(property "Dist" "LCSC"
 			(at 60.96 50.8 0)
 			(effects
@@
 			)
 		)
-		(property "Role" "On-board thermistor"
+		(property "Dist #" "C525660"
 			(at 60.96 38.1 0)
 			(effects
@@
 			)
 		)
-		(property "Part Number" " SDNT1608X103F3435FTF"
+		(property "Mfr" " Sunlord"
 			(at 60.96 38.1 0)
 			(effects
+				(font
+					(size 1.27 1.27)
+				)
+				(hide yes)
+			)
+		)
+		(property "Mfr #" "SDNT1608X103F3435FTF"
+			(at 60.96 38.1 0)
+			(effects
+				(font
+					(size 1.27 1.27)
+				)
+				(hide yes)
+			)
+		)
+		(property "Dist" "LCSC"
+			(at 60.96 38.1 0)
+			(effects
