File: balance.kicad_sch (KiCad schematic)
At the start: 5 parts, among them Q1 IRLML0060

Commit message: schematic: Update to new symbol library
Parts:
- Q1: symbol bms:IRLML0060 -> yfs:IRLML0060
Changed lines of the file:
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@@
 	)
 	(symbol
-		(lib_id "bms:IRLML0060")
+		(lib_id "yfs:IRLML0060")
 		(at 129.54 62.23 0)
 		(unit 1)
