File: bms_segment.kicad_sch (KiCad schematic)
At the start: 95 parts, among them J1 CELL_TAPS, J2 I2C, J5 SWD, J6 I2C, SW1 SW_Push, U1 LMR516xx, U2 STM32F103C8Tx, U3 ADuM1252, U4 MAX14920, U5 MAX11163, U6 REF61xx, Y1 8M

Commit message: bom: Remove spaces from part numbers
Parts:
- C39, C40: Dist # C97954 -> C97954
- U5: Dist # 700-MAX11163EUB+ -> 700-MAX11163EUB+
Changed lines of the file:
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@@
 			)
 		)
-		(property "Dist #" "700-MAX11163EUB+ "
+		(property "Dist #" "700-MAX11163EUB+"
 			(at 181.61 144.78 0)
 			(effects
@@
 			)
 		)
-		(property "Dist #" "C97954 "
+		(property "Dist #" "C97954"
 			(at 217.17 129.54 0)
 			(effects
@@
 			)
 		)
-		(property "Dist #" "C97954 "
+		(property "Dist #" "C97954"
 			(at 226.06 129.54 0)
 			(effects
